Commit message: update

File: src/lerobot_description/urdf/so101.urdf.xacro (robot description, xacro)
@@ -4,3 +4,66 @@
     <xacro:include filename="$(find lerobot_description)/urdf/so101_gazebo.xacro" />
     <xacro:include filename="$(find lerobot_description)/urdf/so101_ros2_control.xacro" />
+    <!-- Add depth camera to the robot -->
+    <link name="camera_link">
+        <visual>
+            <origin xyz="0 0 0" rpy="0 0 0"/>
+            <geometry>
+                <box size="0.1 0.1 0.1"/>
+            </geometry>
+            <material name="camera_material">
+                <color rgba="0.8 0.8 0.8 1"/>
+            </material>
+        </visual>
+        <collision>
+            <origin xyz="0 0 0" rpy="0 0 0"/>
+            <geometry>
+                <box size="0.1 0.1 0.1"/>
+            </geometry>
+        </collision>
+        <inertial>
+            <mass value="0.1"/>
+            <inertia ixx="0.000166667" ixy="0" ixz="0" iyy="0.000166667" iyz="0" izz="0.000166667"/>
+        </inertial>
+    </link>
+    <!-- Joint connecting camera to base -->
+    <joint name="camera_joint" type="fixed">
+        <parent link="base"/>
+        <child link="camera_link"/>
+        <origin xyz="0.0 -0.8 0.3" rpy="0 0 0"/>
+    </joint>
+    <!-- Gazebo sensor configuration -->
+    <gazebo reference="camera_link">
+        <!-- RGB Camera sensor -->
+        <sensor type="camera" name="rgb_camera">
+            <update_rate>30</update_rate>
+            <camera>
+                <horizontal_fov>1.047</horizontal_fov>
+                <image>
+                    <width>640</width>
+                    <height>480</height>
+                    <format>B8G8R8</format>
+                </image>
+                <clip>
+                    <near>0.1</near>
+                    <far>10.0</far>
+                </clip>
+            </camera>
+        </sensor>
+        <!-- Depth Camera sensor -->
+        <sensor type="depth" name="depth_camera">
+            <update_rate>30</update_rate>
+            <camera>
+                <horizontal_fov>1.047</horizontal_fov>
+                <image>
+                    <width>640</width>
+                    <height>480</height>
+                    <format>R_FLOAT32</format>
+                </image>
+                <clip>
+                    <near>0.1</near>
+                    <far>10.0</far>
+                </clip>
+            </camera>
+        </sensor>
+    </gazebo>
 </robot>
